File: hardware/kicad/focalpoint.kicad_sch (KiCad schematic)
At the start: 101 parts, among them J1 USB4105-GF-A-060, J2 SM02B-SRSS-TB, J3 TC2030-IDC-NL, SW14 B3U-1000P, SW15 B3U-1000P, U1 MDBT50Q-1MV2, U2 TPD2EUSB30DRTR, U3 BQ24074RGTR, U4 TPS63031DSKT, U5 TPS61023DRLR, U6 TPS22918DBVR, U7 SN74AHCT1G125DBVR, U8 AT42QT1010-TSHR, U9 MAX17048G+T10

Commit message: Hardware: add validated six-layer Rev A electrical design
Parts:
- added C35, C36: 10nF, Capacitor_SMD:C_0603_1608Metric, symbol focalpoint:C
- added D15: PESD5V0U2BT,215, Package_TO_SOT_SMD:SOT-23, symbol focalpoint:D_TVS_DUAL_CA
- added R23, R24: 1k, Resistor_SMD:R_0603_1608Metric, symbol focalpoint:R
- added R25: 100k, Resistor_SMD:R_0603_1608Metric, symbol focalpoint:R
- C1, C10, C11, C12, C13, C14, C15, C16, C17, C18, C19, C2, C20, C21, C23, C24, C25, C26, C27, C28, C29, C3, C30, C31, C32, C33, C34, C4, C5, C6, C7, C8, C9: footprint (none) -> Capacitor_SMD:C_0603_1608Metric
- D14: footprint (none) -> Diode_SMD:D_SOD-882
- ENC1: footprint (none) -> Rotary_Encoder:RotaryEncoder_Alps_EC11E-Switch_Vertical_H20mm
- HS1, HS10, HS11, HS12, HS13, HS2, HS3, HS4, HS5, HS6, HS7, HS8, HS9: footprint (none) -> FocalPoint:Kailh_CPG151101S11_Hotswap
- J1: footprint (none) -> Connector_USB:USB_C_Receptacle_GCT_USB4105-xx-A_16P_TopMnt_Horizontal
- J2: footprint (none) -> Connector_JST:JST_SH_SM02B-SRSS-TB_1x02-1MP_P1.00mm_Horizontal
- J3: footprint (none) -> Connector:Tag-Connect_TC2030-IDC-NL_2x03_P1.27mm_Vertical
- JS1: value RKJX21224001 -> RKJXV122400R; footprint (none) -> FocalPoint:Alps_RKJXV122400R
- L1: footprint (none) -> Inductor_SMD:L_Sunlord_SWPA3015S
- L2: footprint (none) -> Inductor_SMD:L_Sunlord_MWSA0402S
- LED1, LED10, LED11, LED12, LED13, LED2, LED3, LED4, LED5, LED6, LED7, LED8, LED9: footprint (none) -> LED_SMD:LED_SK6812MINI-E_3.2x2.8mm_P1.5mm_ReverseMount
- R1, R10, R11, R12, R13, R14, R15, R16, R17, R18, R19, R2, R20, R21, R22, R3, R4, R5, R6, R7, R8, R9: footprint (none) -> Resistor_SMD:R_0603_1608Metric
- SW14, SW15: footprint (none) -> Button_Switch_SMD:SW_SPST_B3U-1000P
- U1: footprint (none) -> RF_Module:Raytac_MDBT50Q
- U2: footprint (none) -> Package_TO_SOT_SMD:Texas_DRT-3
- U3: footprint (none) -> Package_DFN_QFN:VQFN-16-1EP_3x3mm_P0.5mm_EP1.68x1.68mm_ThermalVias
- U4: footprint (none) -> Package_SON:WSON-10-1EP_2.5x2.5mm_P0.5mm_EP1.2x2mm_ThermalVias
- U5: footprint (none) -> Package_TO_SOT_SMD:SOT-563
- U6, U8: footprint (none) -> Package_TO_SOT_SMD:SOT-23-6
- U7: footprint (none) -> Package_TO_SOT_SMD:SOT-23-5
- U9: footprint (none) -> Package_DFN_QFN:TDFN-8-1EP_2x2mm_P0.5mm_EP0.8x1.2mm
Connections:
- net +3V3: now also U1.28 (VDD), U3.5 (EN2), U4.1 (VOUT), U4.10 (FB), U8.5 (VDD), R25.1; no longer U1.1 (VDD), U3.12 (EN2), U4.4 (VOUT), U4.5 (FB), U8.1 (VDD)
- net +5V: now also U5.6 (VOUT), U7.5 (VCC); no longer L2.2, U5.3 (VOUT), U7.1 (VCC)
- net +5V_LED: now also U6.5 (QOD), U6.6 (VOUT); no longer U6.2 (VOUT), U6.4 (QOD)
- net +BAT: now also U3.2 (BAT), U9.2 (CELL), U9.3 (CELL_VDD); no longer U9.1 (CELL_VDD)
- net BB_L1: now also U4.4 (L1); no longer U4.2 (L1)
- net BB_L2: now also U4.2 (L2); no longer U4.3 (L2)
- net BOOST_EN: now also U1.6 (BOOST_EN), U5.2 (EN); no longer U1.25 (BOOST_EN), U5.5 (EN)
- net BOOST_FB: now also U5.1 (FB); no longer U5.4 (FB)
- net BQ_ILIM: now also U3.12 (ILIM); no longer U3.5 (ILIM)
- net BQ_ISET: now also U3.16 (ISET); no longer U3.4 (ISET)
- net BQ_ITERM: now also U3.15 (ITERM); no longer U3.6 (ITERM)
- net BQ_TMR: now also U3.14 (TMR); no longer U3.7 (TMR)
- net BQ_TS: now also U3.1 (TS); no longer U3.8 (TS)
- net CC1: now also D15.1 (K1)
- net CC2: now also D15.2 (K2)
- net CHG_STAT: now also U1.29 (CHG_STAT); no longer U1.26 (CHG_STAT)
- net DFU: now also U1.37 (DFU_P013); no longer U1.35 (DFU_P013)
- net ENC_A: now also ENC1.A, U1.41 (ENC_A); no longer ENC1.1 (A), U1.19 (ENC_A)
- net ENC_B: now also ENC1.B, U1.42 (ENC_B); no longer ENC1.2 (B), U1.20 (ENC_B)
- net ENC_SW: now also ENC1.S1 (SW1), U1.44 (ENC_SW); no longer ENC1.4 (SW1), U1.21 (ENC_SW)
- net FG_ALRT: now also U1.48 (FG_ALRT), R25.2; no longer U1.30 (FG_ALRT)
- net FG_SCL: now also U1.14 (FG_SCL), U9.7 (SCL); no longer U1.29 (FG_SCL), U9.4 (SCL)
- net FG_SDA: now also U1.8 (FG_SDA), U9.8 (SDA); no longer U1.28 (FG_SDA), U9.3 (SDA)
- net GND: now also ENC1.C (COMMON), ENC1.S2 (SW2), J1.SH (SHIELD), U1.1 (GND), U1.15 (GND15), U1.33 (GND33), U1.55 (GND55), U2.3 (GND), U3.17 (VSS), U3.4 (CE), U3.6 (EN1), U3.8 (VSS), U4.11 (EP), U4.3 (PGND), U4.9 (GND), U5.4 (GND), U6.2 (GND), U7.3 (GND), U8.6 (SYNC_MODE), U9.1 (CTG), U9.4 (GND), U9.6 (QSTRT), U9.9 (EP), C35.2, C36.2, D15.3 (A); no longer ENC1.3 (COMMON), ENC1.5 (SW2), U2.1 (GND), U3.11 (EN1), U3.13 (VSS), U4.8 (GND), U5.6 (GND), U6.6 (GND), U7.5 (GND), U9.2 (GND)
- net JOY_SW: now also U1.38 (JOY_SW); no longer U1.18 (JOY_SW)
- net JOY_X: now also R23.1; no longer U1.16 (JOY_X_AIN0)
- net JOY_Y: now also R24.1; no longer U1.17 (JOY_Y_AIN1)
- net KEY1: now also U1.47 (KEY1); no longer U1.3 (KEY1)
- net KEY10: now also U1.26 (KEY10); no longer U1.12 (KEY10)
- net KEY11: now also U1.3 (KEY11); no longer U1.13 (KEY11)
- net KEY12: now also U1.4 (KEY12); no longer U1.14 (KEY12)
- net KEY13: now also U1.5 (KEY13); no longer U1.15 (KEY13)
- net KEY2: now also U1.61 (KEY2); no longer U1.4 (KEY2)
- net KEY3: now also U1.50 (KEY3); no longer U1.5 (KEY3)
- net KEY4: now also U1.60 (KEY4); no longer U1.6 (KEY4)
- net KEY5: now also U1.56 (KEY5); no longer U1.7 (KEY5)
- net KEY6: now also U1.59 (KEY6); no longer U1.8 (KEY6)
- net KEY7: now also U1.57 (KEY7); no longer U1.9 (KEY7)
- net KEY8: now also U1.58 (KEY8); no longer U1.10 (KEY8)
- net KEY9: now also U1.25 (KEY9); no longer U1.11 (KEY9)
- net L2_SW: now also U5.5 (SW); no longer U5.2 (SW)
- net PGOOD: now also U1.36 (PGOOD), U3.7 (nPGOOD); no longer U1.27 (PGOOD), U3.10 (nPGOOD)
- net RESET: now also U1.40 (nRESET_P018); no longer U1.36 (nRESET_P018)
- net RGB_DATA: now also U1.22 (RGB_DATA); no longer U1.23 (RGB_DATA)
- net RGB_OE_N: now also U7.1 (OE); no longer U7.3 (OE)
- net SWDCLK: now also U1.53 (SWDCLK); no longer U1.34 (SWDCLK)
- net SWDIO: now also U1.51 (SWDIO); no longer U1.33 (SWDIO)
- net SYS: now also L2.2, U3.10 (SYS), U3.11 (OUT), U4.5 (VIN), U4.8 (VINA), U5.3 (VIN); no longer U3.2 (SYS), U4.1 (VIN), U5.1 (VIN)
- net TOUCH_OUT: now also U1.39 (TOUCH_OUT); no longer U1.22 (TOUCH_OUT)
- net TOUCH_RAW: now also U8.1 (OUT); no longer U8.5 (OUT)
- net U6_CT: now also U6.4 (CT); no longer U6.5 (CT)
- net USB_DN_ESD: now also U1.34 (USB_DN), U2.2 (D-); no longer U2.3 (IO2)
- net USB_DP_ESD: now also U1.35 (USB_DP), U2.1 (D+); no longer U2.2 (IO1)
- net VBUS: now also C26.1, U1.32 (VBUS), U3.13 (IN); no longer U2.6 (VBUS), U3.1 (IN)
- removed net BQ_VDPM: C26.1, U3.14 (VDPM)
- removed net USB_DN: U1.32 (USB_DN), U2.5 (OUT2)
- removed net USB_DP: U1.31 (USB_DP), U2.4 (OUT1)
- new net JOY_X_FILT: C35.1, R23.2, U1.11 (JOY_X_AIN0)
- new net JOY_Y_FILT: C36.1, R24.2, U1.9 (JOY_Y_AIN1)
