File: hardware/kicad/focalpoint.kicad_sch (KiCad schematic)
At the start: 107 parts, among them J1 USB4105-GF-A-060, J2 SM02B-SRSS-TB, J3 TC2030-IDC-NL, SW14 B3U-1000P, SW15 B3U-1000P, U1 MDBT50Q-1MV2, U2 TPD2EUSB30DRTR, U3 BQ24074RGTR, U4 TPS63031DSKT, U5 TPS61023DRLR, U6 TPS22918DBVR, U7 SN74AHCT1G125DBVR, U8 AT42QT1010-TSHR, U9 MAX17048G+T10

Commit message: Hardware: organize Rev A schematic into functional sheets
Split the verified flat capture into power, signals, and peripherals sheets,
preserve the locked reference, and package hierarchy validation evidence.

Co-Authored-By: Claude Opus 4.8 <noreply@anthropic.com>
Parts:
- removed BT1: ASR00012, symbol focalpoint:BT_CELL
- removed C1, C10, C11, C12, C13, C14, C15, C16, C17, C18, C19, C2, C20, C21, C3, C4, C5, C6, C7, C8, C9: 100nF, Capacitor_SMD:C_0603_1608Metric, symbol focalpoint:C
- removed C23, C24, C25: 4.7uF, Capacitor_SMD:C_0603_1608Metric, symbol focalpoint:C
- removed C26: 1uF, Capacitor_SMD:C_0603_1608Metric, symbol focalpoint:C
- removed C27, C28, C29, C30: 10uF, Capacitor_SMD:C_0603_1608Metric, symbol focalpoint:C
- removed C31, C32: 22uF, Capacitor_SMD:C_0603_1608Metric, symbol focalpoint:C
- removed C33: 220pF, Capacitor_SMD:C_0603_1608Metric, symbol focalpoint:C
- removed C34, C35, C36: 10nF, Capacitor_SMD:C_0603_1608Metric, symbol focalpoint:C
- removed D14: PESD5V0S1UL, Diode_SMD:D_SOD-882, symbol focalpoint:D_TVS
- removed D15: PESD5V0U2BT,215, Package_TO_SOT_SMD:SOT-23, symbol focalpoint:D_TVS_DUAL_CA
- removed ENC1: EC11E15244G1, Rotary_Encoder:RotaryEncoder_Alps_EC11E-Switch_Vertical_H20mm, symbol focalpoint:ENC_EC11
- removed HS1, HS10, HS11, HS12, HS13, HS2, HS3, HS4, HS5, HS6, HS7, HS8, HS9: CPG151101S11, FocalPoint:Kailh_CPG151101S11_Hotswap, symbol focalpoint:SW2
- removed J1: USB4105-GF-A-060, Connector_USB:USB_C_Receptacle_GCT_USB4105-xx-A_16P_TopMnt_Horizontal, symbol focalpoint:J_USBC
- removed J2: SM02B-SRSS-TB, Connector_JST:JST_SH_SM02B-SRSS-TB_1x02-1MP_P1.00mm_Horizontal, symbol focalpoint:J_BATT
- removed J3: TC2030-IDC-NL, Connector:Tag-Connect_TC2030-IDC-NL_2x03_P1.27mm_Vertical, symbol focalpoint:J_SWD
- removed JS1: RKJXV122400R, FocalPoint:Alps_RKJXV122400R, symbol focalpoint:JOY_ALPS
- removed L1: 1.5uH, Inductor_SMD:L_Sunlord_SWPA3015S, symbol focalpoint:L
- removed L2: 1.0uH, Inductor_SMD:L_Sunlord_MWSA0402S, symbol focalpoint:L
- removed LED1, LED10, LED11, LED12, LED13, LED2, LED3, LED4, LED5, LED6, LED7, LED8, LED9: SK6812MINI-E, LED_SMD:LED_SK6812MINI-E_3.2x2.8mm_P1.5mm_ReverseMount, symbol focalpoint:LED4
- removed R1, R2: 5.1k, Resistor_SMD:R_0603_1608Metric, symbol focalpoint:R
- removed R10, R11, R12, R13, R25: 100k, Resistor_SMD:R_0603_1608Metric, symbol focalpoint:R
- removed R14, R15, R16, R17: 10k, Resistor_SMD:R_0603_1608Metric, symbol focalpoint:R
- removed R18, R19: 4.7k, Resistor_SMD:R_0603_1608Metric, symbol focalpoint:R
- removed R20, R21, R23, R24: 1k, Resistor_SMD:R_0603_1608Metric, symbol focalpoint:R
- removed R22: 33R, Resistor_SMD:R_0603_1608Metric, symbol focalpoint:R
- removed R3, R4: 22R DNP, Resistor_SMD:R_0603_1608Metric, symbol focalpoint:R
- removed R5: 2.21k, Resistor_SMD:R_0603_1608Metric, symbol focalpoint:R
- removed R6: 3.09k, Resistor_SMD:R_0603_1608Metric, symbol focalpoint:R
- removed R7: 2.94k, Resistor_SMD:R_0603_1608Metric, symbol focalpoint:R
- removed R8: 46.4k, Resistor_SMD:R_0603_1608Metric, symbol focalpoint:R
- removed R9: 732k, Resistor_SMD:R_0603_1608Metric, symbol focalpoint:R
- removed SW14, SW15: B3U-1000P, Button_Switch_SMD:SW_SPST_B3U-1000P, symbol focalpoint:SW2
- removed U1: MDBT50Q-1MV2, RF_Module:Raytac_MDBT50Q, symbol focalpoint:U1_MODULE
- removed U2: TPD2EUSB30DRTR, Package_TO_SOT_SMD:Texas_DRT-3, symbol focalpoint:U2_ESD
- removed U3: BQ24074RGTR, Package_DFN_QFN:VQFN-16-1EP_3x3mm_P0.5mm_EP1.68x1.68mm_ThermalVias, symbol focalpoint:U3_CHARGER
- removed U4: TPS63031DSKT, Package_SON:WSON-10-1EP_2.5x2.5mm_P0.5mm_EP1.2x2mm_ThermalVias, symbol focalpoint:U4_BUCKBOOST
- removed U5: TPS61023DRLR, Package_TO_SOT_SMD:SOT-563, symbol focalpoint:U5_BOOST
- removed U6: TPS22918DBVR, Package_TO_SOT_SMD:SOT-23-6, symbol focalpoint:U6_LOADSW
- removed U7: SN74AHCT1G125DBVR, Package_TO_SOT_SMD:SOT-23-5, symbol focalpoint:U7_BUFFER
- removed U8: AT42QT1010-TSHR, Package_TO_SOT_SMD:SOT-23-6, symbol focalpoint:U8_TOUCH
- removed U9: MAX17048G+T10, Package_DFN_QFN:TDFN-8-1EP_2x2mm_P0.5mm_EP0.8x1.2mm, symbol focalpoint:U9_FUELGAUGE
Connections:
- no-connect marks 4 -> 0
Other:
- added sheet Controller and Signals (focalpoint_signals.kicad_sch)
- added sheet Inputs, RGB, and Peripherals (focalpoint_peripherals.kicad_sch)
- added sheet Power Electronics (focalpoint_power.kicad_sch)
- title: (none) -> FocalPoint Rev A — System Hierarchy
